Commit message: Sockel added for sim config

File: code/manipulator_description/urdf/manipulator_gz.urdf.xacro (robot description, xacro)
@@ -15,4 +15,6 @@
   <!-- import Scene Objects macro -->
   <xacro:include filename="$(find manipulator_description)/urdf/schrankregal.xacro"/>
+  <!-- import UR Sockel macro -->
+  <xacro:include filename="$(find manipulator_description)/urdf/ur_sockel.xacro"/>
   <!-- possible 'ur_type' values: ur3, ur3e, ur5, ur5e, ur7e, ur10, ur10e, ur12e, ur16e, ur15, ur20, ur30 -->
   <!-- the default value should raise an error in case this was called without defining the type -->
@@ -59,4 +61,11 @@
     <child link="ground_plane"/>
   </joint>
+  <!-- UR Sockel -->
+  <xacro:ur_sockel
+    name="ur_sockel"
+    parent_link="world"
+    xyz="0 0 0"
+    rpy="0 0 0">
+  </xacro:ur_sockel>
   <!-- scene -->
   <xacro:schrankregal
@@ -93,5 +102,5 @@
     safety_k_position="$(arg safety_k_position)"
     force_abs_paths="true">
-    <origin xyz="0 0 0" rpy="0 0 0" />
+    <origin xyz="0 0 0.07" rpy="0 0 0" />
   </xacro:ur_robot>
   <xacro:ur_realsense_mount

File: code/manipulator_ur_moveit_config/srdf/ur_macro.srdf.xacro (robot description, xacro)
@@ -53,4 +53,9 @@
     <disable_collisions link1="wrist_1_link" link2="wrist_3_link" reason="Never" />
     <disable_collisions link1="wrist_2_link" link2="wrist_3_link" reason="Adjacent" />
+    <!-- disable sockel collisions -->
+    <disable_collisions link1="ur_sockel_link" link2="base_link" reason="Adjacent" />
+    <disable_collisions link1="ur_sockel_link" link2="ground_plane" reason="Adjacent" />
+    <disable_collisions link1="ur_sockel_link" link2="unten_schrankregal_link" reason="Adjacent" />
+    <disable_collisions link1="ur_sockel_link" link2="base_link_inertia" reason="Adjacent" />
   </xacro:macro>
 </robot>
