Commit message: Merge sim and hardware urdf

File: code/manipulator_description/urdf/manipulator.urdf.xacro (robot description, xacro)
@@ -1,9 +1,16 @@
 <?xml version="1.0" encoding="utf-8"?>
 <robot xmlns:xacro="http://wiki.ros.org/xacro" name="ur5e">
+  <xacro:arg name="use_mock_hardware" default="false" />
+  <xacro:property name="use_mock_hardware" default="$(arg use_mock_hardware)"/>
   <!-- import ur5 macro -->
   <xacro:include filename="$(find ur_description)/urdf/ur_macro.xacro"/>
   <!-- import ur5 ROS2 control macro -->
-  <xacro:include filename="$(find ur_robot_driver)/urdf/ur.ros2_control.xacro"/>
-  <xacro:include filename="$(find ur_description)/urdf/inc/ur_transmissions.xacro" />
+  <xacro:if value="${use_mock_hardware}">
+    <xacro:include filename="$(find ur_simulation_gz)/urdf/ur_gz.ros2_control.xacro" />
+  </xacro:if>
+  <xacro:unless value="${use_mock_hardware}">
+    <xacro:include filename="$(find ur_robot_driver)/urdf/ur.ros2_control.xacro"/>
+    <xacro:include filename="$(find ur_description)/urdf/inc/ur_transmissions.xacro" />
+  </xacro:unless>
   <!-- import Mia Hand macro -->
   <xacro:include filename="$(find mia_hand_description)/urdf/mia_hand.urdf.xacro"/>
@@ -16,4 +23,6 @@
   <!-- import Scene Objects macro -->
   <xacro:include filename="$(find manipulator_description)/urdf/schrankregal.xacro"/>
+  <!-- import UR Sockel macro -->
+  <xacro:include filename="$(find manipulator_description)/urdf/ur_sockel.xacro"/>
   <!-- ur5 parameters -->
   <!-- possible 'ur_type' values: ur3, ur3e, ur5, ur5e, ur7e, ur10, ur10e, ur12e, ur16e, ur15, ur20, ur30 -->
@@ -29,28 +38,31 @@
   <xacro:arg name="safety_pos_margin" default="0.15"/>
   <xacro:arg name="safety_k_position" default="20"/>
-  <xacro:arg name="headless_mode" default="false" />
-  <xacro:arg name="robot_ip" default="0.0.0.0"/>
-  <xacro:arg name="script_filename" default=""/>
-  <xacro:arg name="output_recipe_filename" default=""/>
-  <xacro:arg name="input_recipe_filename" default=""/>
-  <xacro:arg name="reverse_ip" default="0.0.0.0"/>
-  <xacro:arg name="script_command_port" default="50004"/>
-  <xacro:arg name="reverse_port" default="50001"/>
-  <xacro:arg name="script_sender_port" default="50002"/>
-  <xacro:arg name="trajectory_port" default="50003"/>
-  <!--   tool communication related parameters-->
-  <xacro:arg name="use_tool_communication" default="false" />
-  <xacro:arg name="tool_voltage" default="0" />
-  <xacro:arg name="tool_parity" default="0" />
-  <xacro:arg name="tool_baud_rate" default="115200" />
-  <xacro:arg name="tool_stop_bits" default="1" />
-  <xacro:arg name="tool_rx_idle_chars" default="1.5" />
-  <xacro:arg name="tool_tx_idle_chars" default="3.5" />
-  <xacro:arg name="tool_device_name" default="/tmp/ttyUR" />
-  <xacro:arg name="tool_tcp_port" default="54321" />
+  <xacro:unless value="${use_mock_hardware}">
+    <!-- Robot hardware parameters -->
+    <xacro:arg name="headless_mode" default="false" />
+    <xacro:arg name="robot_ip" default="0.0.0.0"/>
+    <xacro:arg name="script_filename" default=""/>
+    <xacro:arg name="output_recipe_filename" default=""/>
+    <xacro:arg name="input_recipe_filename" default=""/>
+    <xacro:arg name="reverse_ip" default="0.0.0.0"/>
+    <xacro:arg name="script_command_port" default="50004"/>
+    <xacro:arg name="reverse_port" default="50001"/>
+    <xacro:arg name="script_sender_port" default="50002"/>
+    <xacro:arg name="trajectory_port" default="50003"/>
+    <!--   tool communication related parameters-->
+    <xacro:arg name="use_tool_communication" default="false" />
+    <xacro:arg name="tool_voltage" default="0" />
+    <xacro:arg name="tool_parity" default="0" />
+    <xacro:arg name="tool_baud_rate" default="115200" />
+    <xacro:arg name="tool_stop_bits" default="1" />
+    <xacro:arg name="tool_rx_idle_chars" default="1.5" />
+    <xacro:arg name="tool_tx_idle_chars" default="3.5" />
+    <xacro:arg name="tool_device_name" default="/tmp/ttyUR" />
+    <xacro:arg name="tool_tcp_port" default="54321" />
+  </xacro:unless>
   <!-- Simulation parameters -->
-  <xacro:arg name="use_mock_hardware" default="false" />
   <xacro:arg name="mock_sensor_commands" default="false" />
   <xacro:arg name="simulation_controllers" default="" />
+  <xacro:arg name="ros_namespace" default="" />
   <!-- initial position for simulations (Mock Hardware, Gazebo, Ignition) -->
   <xacro:arg name="initial_positions_file" default="$(find ur_description)/config/initial_positions.yaml"/>
@@ -87,4 +99,11 @@
     <child link="ground_plane"/>
   </joint>
+  <!-- UR Sockel -->
+  <xacro:ur_sockel
+    name="ur_sockel"
+    parent_link="world"
+    xyz="0 0 0"
+    rpy="0 0 0">
+  </xacro:ur_sockel>
   <!-- scene -->
   <xacro:schrankregal
@@ -110,7 +129,7 @@
   <!-- arm -->
   <xacro:ur_robot
+    parent="world"
     name="$(arg ur_type)"
     tf_prefix="$(arg tf_prefix)"
-    parent="world"
     joint_limits_parameters_file="$(arg joint_limit_params)"
     kinematics_parameters_file="$(arg kinematics_params)"
@@ -119,6 +138,7 @@
     safety_limits="$(arg safety_limits)"
     safety_pos_margin="$(arg safety_pos_margin)"
-    safety_k_position="$(arg safety_k_position)">
-     <origin xyz="0 0 0" rpy="0 0 0" />          <!-- position robot in the world -->
+    safety_k_position="$(arg safety_k_position)"
+    force_abs_paths="true">
+    <origin xyz="0 0 0.07" rpy="0 0 0" /> <!-- position robot in the world -->
   </xacro:ur_robot>
   <xacro:ur_realsense_mount
@@ -131,5 +151,5 @@
     laterality="$(arg laterality)"
     joint_limits_config_file="$(arg joint_limits_config_file)"
-    parent="tool0"
+    parent="ur_realsense_mount_link"
     prefix="$(arg prefix)">
     <xacro:if value="${'right' == '$(arg laterality)'}">
@@ -140,6 +160,6 @@
     </xacro:if>
   </xacro:mia_hand>
-   <!-- RealSense D435 Camera -->
-  <xacro:sensor_d435
+  <!-- RealSense D435 Camera -->
+  <!-- <xacro:sensor_d435
       name="camera_tower"
       parent="base_link"
@@ -148,6 +168,6 @@
       use_mesh="true">
     <origin xyz="0 0 1.30" rpy="0 1 1"/>
-  </xacro:sensor_d435>
-    <!-- RealSense D435 Camera Tool-->
+  </xacro:sensor_d435> -->
+  <!-- RealSense D435 Camera Tool-->
   <xacro:sensor_d435
       name="camera_gripper"
@@ -158,33 +178,74 @@
     <origin xyz="0 0.110 0.012" rpy="0 -1.57 -1.57"/>
   </xacro:sensor_d435>
+  <xacro:if value="${use_mock_hardware}">
+    <!-- Gazebo specific elements -->
+    <gazebo reference="world"></gazebo>
+    <gazebo>
+      <plugin filename="gz_ros2_control-system" name="gz_ros2_control::GazeboSimROS2ControlPlugin">
+        <parameters>$(arg simulation_controllers)</parameters>
+        <ros>
+          <namespace>$(arg ros_namespace)</namespace>
+        </ros>
+      </plugin>
+    </gazebo>
+    <!-- <gazebo reference="camera_depth_frame">
+      <sensor name="rgbd_camera" type="rgbd_camera">
+        <always_on>true</always_on>
+        <update_rate>5</update_rate>
+        <visualize>true</visualize>
+        <camera>
+          <horizontal_fov>1</horizontal_fov>
+          <image>
+            <width>640</width>
+            <height>480</height>
+            <format>R8G8B8</format>
+          </image>
+          <clip>
+            <near>0.05</near>
+            <far>3.0</far>
+          </clip>
+        </camera>
+        <topic>/rgbd_camera</topic>
+      </sensor>
+    </gazebo> -->
+  </xacro:if>
   <!-- ros2 control instance -->
-  <xacro:ur_ros2_control
-    name="$(arg ur_type)"
-    tf_prefix="$(arg tf_prefix)"
-    kinematics_parameters_file="$(arg kinematics_params)"
-    transmission_hw_interface="$(arg transmission_hw_interface)"
-    use_mock_hardware="$(arg use_mock_hardware)"
-    mock_sensor_commands="$(arg mock_sensor_commands)"
-    headless_mode="$(arg headless_mode)"
-    initial_positions="${xacro.load_yaml(initial_positions_file)}"
-    use_tool_communication="$(arg use_tool_communication)"
-    tool_voltage="$(arg tool_voltage)"
-    tool_parity="$(arg tool_parity)"
-    tool_baud_rate="$(arg tool_baud_rate)"
-    tool_stop_bits="$(arg tool_stop_bits)"
-    tool_rx_idle_chars="$(arg tool_rx_idle_chars)"
-    tool_tx_idle_chars="$(arg tool_tx_idle_chars)"
-    tool_device_name="$(arg tool_device_name)"
-    tool_tcp_port="$(arg tool_tcp_port)"
-    robot_ip="$(arg robot_ip)"
-    script_filename="$(arg script_filename)"
-    output_recipe_filename="$(arg output_recipe_filename)"
-    input_recipe_filename="$(arg input_recipe_filename)"
-    reverse_ip="$(arg reverse_ip)"
-    script_command_port="$(arg script_command_port)"
-    reverse_port="$(arg reverse_port)"
-    script_sender_port="$(arg script_sender_port)"
-    trajectory_port="$(arg trajectory_port)"
-  />
+  <xacro:if value="${use_mock_hardware}">
+    <xacro:ur_ros2_control
+      name="$(arg ur_type)"
+      tf_prefix="$(arg tf_prefix)"
+      transmission_hw_interface="$(arg transmission_hw_interface)"
+    />
+  </xacro:if>
+  <xacro:unless value="${use_mock_hardware}">
+    <xacro:ur_ros2_control
+      name="$(arg ur_type)"
+      tf_prefix="$(arg tf_prefix)"
+      kinematics_parameters_file="$(arg kinematics_params)"
+      transmission_hw_interface="$(arg transmission_hw_interface)"
+      use_mock_hardware="$(arg use_mock_hardware)"
+      mock_sensor_commands="$(arg mock_sensor_commands)"
+      headless_mode="$(arg headless_mode)"
+      initial_positions="${xacro.load_yaml(initial_positions_file)}"
+      use_tool_communication="$(arg use_tool_communication)"
+      tool_voltage="$(arg tool_voltage)"
+      tool_parity="$(arg tool_parity)"
+      tool_baud_rate="$(arg tool_baud_rate)"
+      tool_stop_bits="$(arg tool_stop_bits)"
+      tool_rx_idle_chars="$(arg tool_rx_idle_chars)"
+      tool_tx_idle_chars="$(arg tool_tx_idle_chars)"
+      tool_device_name="$(arg tool_device_name)"
+      tool_tcp_port="$(arg tool_tcp_port)"
+      robot_ip="$(arg robot_ip)"
+      script_filename="$(arg script_filename)"
+      output_recipe_filename="$(arg output_recipe_filename)"
+      input_recipe_filename="$(arg input_recipe_filename)"
+      reverse_ip="$(arg reverse_ip)"
+      script_command_port="$(arg script_command_port)"
+      reverse_port="$(arg reverse_port)"
+      script_sender_port="$(arg script_sender_port)"
+      trajectory_port="$(arg trajectory_port)"
+    />
+  </xacro:unless>
   <!-- mia hand ros2 control instance -->
   <xacro:mia_hand_ros2_control

File: code/manipulator_description/urdf/manipulator_gz.urdf.xacro (robot description, xacro)
@@ -1,3 +1,3 @@
-<?xml version="1.0"?>
+<?xml version="1.0" encoding="utf-8"?>
 <robot xmlns:xacro="http://wiki.ros.org/xacro" name="ur5e">
   <!-- import ur5 macro -->
@@ -17,4 +17,5 @@
   <!-- import UR Sockel macro -->
   <xacro:include filename="$(find manipulator_description)/urdf/ur_sockel.xacro"/>
+  <!-- ur5 parameters -->
   <!-- possible 'ur_type' values: ur3, ur3e, ur5, ur5e, ur7e, ur10, ur10e, ur12e, ur16e, ur15, ur20, ur30 -->
   <!-- the default value should raise an error in case this was called without defining the type -->
@@ -29,6 +30,12 @@
   <xacro:arg name="safety_pos_margin" default="0.15"/>
   <xacro:arg name="safety_k_position" default="20"/>
+  <!-- Simulation parameters -->
+  <xacro:arg name="mock_sensor_commands" default="false" />
   <xacro:arg name="simulation_controllers" default="" />
   <xacro:arg name="ros_namespace" default="" />
+  <!-- initial position for simulations (Mock Hardware, Gazebo, Ignition) -->
+  <xacro:arg name="initial_positions_file" default="$(find ur_description)/config/initial_positions.yaml"/>
+  <!-- convert to property to use substitution in function -->
+  <xacro:property name="initial_positions_file" default="$(arg initial_positions_file)"/>
   <!-- mia hand parameters -->
   <xacro:arg name="serial_port" default="/dev/ttyUSB0"/>
@@ -102,5 +109,5 @@
     safety_k_position="$(arg safety_k_position)"
     force_abs_paths="true">
-    <origin xyz="0 0 0.07" rpy="0 0 0" />
+    <origin xyz="0 0 0.07" rpy="0 0 0" /> <!-- position robot in the world -->
   </xacro:ur_robot>
   <xacro:ur_realsense_mount
@@ -122,6 +129,6 @@
     </xacro:if>
   </xacro:mia_hand>
-   <!-- RealSense D435 Camera -->
-  <xacro:sensor_d435
+  <!-- RealSense D435 Camera -->
+  <!-- <xacro:sensor_d435
       name="camera"
       parent="base_link"
@@ -130,7 +137,7 @@
       use_mesh="true">
     <origin xyz="0.35 -0.35 0.57" rpy="0 0 2.35619"/>
-  </xacro:sensor_d435>
+  </xacro:sensor_d435> -->
   <!-- RealSense D435 Camera Tool-->
-  <!-- <xacro:sensor_d435
+  <xacro:sensor_d435
       name="camera"
       parent="tool0"
@@ -138,6 +145,6 @@
       add_plug="false"
       use_mesh="true">
-    <origin xyz="0 0.135 0.012" rpy="0 -1.57 1.57"/>
-  </xacro:sensor_d435> -->
+    <origin xyz="0 0.110 0.012" rpy="0 -1.57 -1.57"/>
+  </xacro:sensor_d435>
   <!-- Gazebo specific elements -->
   <gazebo reference="world"></gazebo>

File: code/manipulator_ur_moveit_config/srdf/manipulator_macro.srdf.xacro (robot description, xacro)
@@ -87,4 +87,9 @@
     <disable_collisions link1="ur_realsense_mount_link" link2="hand_ee_link" reason="Adjacent"/>
     <disable_collisions link1="ur_realsense_mount_link" link2="camera_gripper_link" reason="Adjacent"/>
+    <!-- disable sockel collisions -->
+    <disable_collisions link1="ur_sockel_link" link2="base_link" reason="Adjacent" />
+    <disable_collisions link1="ur_sockel_link" link2="ground_plane" reason="Adjacent" />
+    <disable_collisions link1="ur_sockel_link" link2="unten_schrankregal_link" reason="Adjacent" />
+    <disable_collisions link1="ur_sockel_link" link2="base_link_inertia" reason="Adjacent" />
   </xacro:macro>
 </robot>

Commit message: Fix hardware launch

File: code/manipulator_description/urdf/manipulator.urdf.xacro (robot description, xacro)
@@ -2,5 +2,5 @@
 <robot xmlns:xacro="http://wiki.ros.org/xacro" name="ur5e">
   <xacro:arg name="use_mock_hardware" default="false" />
-  <xacro:property name="use_mock_hardware" default="$(arg use_mock_hardware)"/>
+  <xacro:property name="use_mock_hardware" value="$(arg use_mock_hardware)"/>
   <!-- import ur5 macro -->
   <xacro:include filename="$(find ur_description)/urdf/ur_macro.xacro"/>

File: code/manipulator_description/urdf/mia_hand.ros2_control.xacro (robot description, xacro)
@@ -13,6 +13,6 @@
       <xacro:if value="${use_mock_hardware}">
         <hardware>
-          <!-- <plugin>mock_components/GenericSystem</plugin> -->
-          <plugin>gz_ros2_control/GazeboSimSystem</plugin>
+          <plugin>mock_components/GenericSystem</plugin>
+          <!-- <plugin>gz_ros2_control/GazeboSimSystem</plugin> -->
         </hardware>
         <joint name="j_thumb_opp">
