Commit message: initial upload

File: code/manipulator_description/urdf/manipulator.urdf.xacro (robot description, xacro)
@@ -1,4 +1,4 @@
 <?xml version="1.0" encoding="utf-8"?>
-<robot xmlns:xacro="http://wiki.ros.org/xacro" name="ur5e">
+<robot xmlns:xacro="http://wiki.ros.org/xacro" name="$(arg ur_type)">
   <xacro:arg name="use_mock_hardware" default="false" />
   <xacro:property name="use_mock_hardware" value="$(arg use_mock_hardware)"/>
@@ -14,9 +14,9 @@
   </xacro:unless>
   <!-- import Mia Hand macro -->
-  <xacro:include filename="$(find mia_hand_description)/urdf/mia_hand.urdf.xacro"/>
+  <xacro:include filename="$(find manipulator_description)/urdf/mia_hand.urdf.xacro"/>
   <!-- import Mia Hand ROS2 control macro -->
   <xacro:include filename="$(find manipulator_description)/urdf/mia_hand.ros2_control.xacro"/>
   <!-- import Camera macro -->
-  <xacro:include filename="$(find realsense2_description)/urdf/_d435.urdf.xacro"/>
+  <xacro:include filename="$(find manipulator_description)/urdf/_d435.urdf.xacro"/>
   <!-- import Realsense Mount macro -->
   <xacro:include filename="$(find manipulator_description)/urdf/ur_realsense_mount.xacro"/>
@@ -24,5 +24,7 @@
   <xacro:include filename="$(find manipulator_description)/urdf/schrankregal.xacro"/>
   <!-- import UR Sockel macro -->
-  <xacro:include filename="$(find manipulator_description)/urdf/ur_sockel.xacro"/>
+  <xacro:include filename="$(find manipulator_description)/urdf/ur_chasis.xacro"/>
+    <!-- import Apollo Base macro -->
+  <xacro:include filename="$(find manipulator_description)/urdf/ranger_air_description.xacro"/>
   <!-- ur5 parameters -->
   <!-- possible 'ur_type' values: ur3, ur3e, ur5, ur5e, ur7e, ur10, ur10e, ur12e, ur16e, ur15, ur20, ur30 -->
@@ -99,11 +101,19 @@
     <child link="ground_plane"/>
   </joint>
-  <!-- UR Sockel -->
-  <xacro:ur_sockel
-    name="ur_sockel"
-    parent_link="world"
+  <!-- Apollo2 Base -->
+  <xacro:ranger_air_description
+    name="ranger_air_description"
+    parent_link="world"
+    xyz="1 1 0"
+    rpy="0 0 0"
+    use_mock_hardware="true">
+  </xacro:ranger_air_description>
+  <!-- UR Chasis -->
+  <xacro:ur_chasis
+    name="ur_chasis"
+    parent_link="ranger_base_link"
     xyz="0 0 0"
     rpy="0 0 0">
-  </xacro:ur_sockel>
+  </xacro:ur_chasis>
   <!-- scene -->
   <xacro:schrankregal
@@ -113,5 +123,4 @@
     rpy="1.571 0 -0.785">
   </xacro:schrankregal>
-  <!-- scene -->
   <xacro:schrankregal
     name="mitte"
@@ -120,5 +129,4 @@
     rpy="1.571 0 -0.785">
   </xacro:schrankregal>
-  <!-- scene -->
   <xacro:schrankregal
     name="oben"
@@ -129,5 +137,5 @@
   <!-- arm -->
   <xacro:ur_robot
-    parent="world"
+    parent="ur_chasis_link"
     name="$(arg ur_type)"
     tf_prefix="$(arg tf_prefix)"
@@ -140,5 +148,5 @@
     safety_k_position="$(arg safety_k_position)"
     force_abs_paths="true">
-    <origin xyz="0 0 0.07" rpy="0 0 0" /> <!-- position robot in the world -->
+    <origin xyz="0 0 1.142" rpy="0 0 0" /> <!-- position robot in the world -->
   </xacro:ur_robot>
   <xacro:ur_realsense_mount
@@ -176,5 +184,5 @@
       add_plug="false"
       use_mesh="true">
-    <origin xyz="0 0.110 0.012" rpy="0 -1.57 -1.57"/>
+    <origin xyz="-0.001 0.102 0.052" rpy="0 1.31 1.57"/>
   </xacro:sensor_d435>
   <xacro:if value="${use_mock_hardware}">

File: code/manipulator_description/urdf/mia_hand.ros2_control.xacro (robot description, xacro)
@@ -5,4 +5,5 @@
     params="name prefix serial_port use_mock_hardware">
     <ros2_control name="${name}" type="system">
+      <!-- Real hardware: echte Mia-Hand über Serial Interface -->
       <xacro:unless value="${use_mock_hardware}">
         <hardware>
@@ -11,40 +12,78 @@
         </hardware>
       </xacro:unless>
+      <!-- Simulation: Mia-Hand-Joints werden von Gazebo / gz_ros2_control bereitgestellt -->
       <xacro:if value="${use_mock_hardware}">
         <hardware>
-          <plugin>mock_components/GenericSystem</plugin>
-          <!-- <plugin>gz_ros2_control/GazeboSimSystem</plugin> -->
+          <plugin>gz_ros2_control/GazeboSimSystem</plugin>
         </hardware>
-        <joint name="j_thumb_opp">
-          <command_interface name="position" />
-          <command_interface name="velocity" />
-          <state_interface name="position" />
-          <state_interface name="velocity" />
-        </joint>
-        <joint name="j_ring_fle"></joint>
-        <joint name="j_little_fle"></joint>
-        <joint name="j_thumb_fle">
-          <command_interface name="position" />
-          <command_interface name="velocity" />
-          <state_interface name="position" />
-          <state_interface name="velocity" />
-        </joint>
-        <joint name="j_index_fle">
-          <command_interface name="position" />
-          <command_interface name="velocity" />
-          <state_interface name="position" />
-          <state_interface name="velocity" />
-        </joint>
-        <joint name="j_mrl_fle">
-          <command_interface name="position" />
-          <command_interface name="velocity" />
-          <state_interface name="position" />
-          <state_interface name="velocity" />
-        </joint>
       </xacro:if>
-      <!-- Extra joints used only for Rviz2 visualization -->
-      <!-- <joint name="j_thumb_opp" />
-      <joint name="j_ring_fle" />
-      <joint name="j_little_fle" /> -->
+      <!-- Thumb opposition joint: nur falls du ihn später auch steuern willst -->
+      <joint name="${prefix}j_thumb_opp">
+        <command_interface name="position">
+          <param name="min">-1.0</param>
+          <param name="max">1.0</param>
+        </command_interface>
+        <command_interface name="velocity">
+          <param name="min">-2.0</param>
+          <param name="max">2.0</param>
+        </command_interface>
+        <state_interface name="position">
+          <param name="initial_value">0.0</param>
+        </state_interface>
+        <state_interface name="velocity">
+          <param name="initial_value">0.0</param>
+        </state_interface>
+      </joint>
+      <!-- Thumb flexion -->
+      <joint name="${prefix}j_thumb_fle">
+        <command_interface name="position">
+          <param name="min">0.0</param>
+          <param name="max">1.2</param>
+        </command_interface>
+        <command_interface name="velocity">
+          <param name="min">-2.0</param>
+          <param name="max">2.0</param>
+        </command_interface>
+        <state_interface name="position">
+          <param name="initial_value">0.0</param>
+        </state_interface>
+        <state_interface name="velocity">
+          <param name="initial_value">0.0</param>
+        </state_interface>
+      </joint>
+      <!-- Index flexion -->
+      <joint name="${prefix}j_index_fle">
+        <command_interface name="position">
+          <param name="min">0.0</param>
+          <param name="max">1.2</param>
+        </command_interface>
+        <command_interface name="velocity">
+          <param name="min">-2.0</param>
+          <param name="max">2.0</param>
+        </command_interface>
+        <state_interface name="position">
+          <param name="initial_value">0.0</param>
+        </state_interface>
+        <state_interface name="velocity">
+          <param name="initial_value">0.0</param>
+        </state_interface>
+      </joint>
+      <!-- Middle / Ring / Little flexion combined -->
+      <joint name="${prefix}j_mrl_fle">
+        <command_interface name="position">
+          <param name="min">0.0</param>
+          <param name="max">1.2</param>
+        </command_interface>
+        <command_interface name="velocity">
+          <param name="min">-2.0</param>
+          <param name="max">2.0</param>
+        </command_interface>
+        <state_interface name="position">
+          <param name="initial_value">0.0</param>
+        </state_interface>
+        <state_interface name="velocity">
+          <param name="initial_value">0.0</param>
+        </state_interface>
+      </joint>
     </ros2_control>
   </xacro:macro>

File: code/manipulator_description/urdf/ur_realsense_mount.xacro (robot description, xacro)
@@ -7,5 +7,5 @@
         <origin xyz="${xyz}" rpy="${rpy}"/>
         <geometry>
-          <mesh filename="package://manipulator_description/meshes/halterung_realsense.stl" scale="0.001 0.001 0.001"/>
+          <mesh filename="file://$(find manipulator_description)/meshes/halterung_realsense.stl" scale="0.001 0.001 0.001"/>
         </geometry>
         <material name="MYBLACK"/>
@@ -14,5 +14,5 @@
         <origin xyz="${xyz}" rpy="${rpy}"/>
         <geometry>
-          <mesh filename="package://manipulator_description/meshes/halterung_realsense.stl" scale="0.001 0.001 0.001"/>
+          <mesh filename="file://$(find manipulator_description)/meshes/halterung_realsense.stl" scale="0.001 0.001 0.001"/>
         </geometry>
       </collision>

File: code/manipulator_ur_moveit_config/srdf/manipulator_macro.srdf.xacro (robot description, xacro)
@@ -47,21 +47,24 @@
       <joint name="wrist_3_joint" value="-0.11" />
     </group_state>
-    <!-- Hand-States (anpassen, falls andere Neutralwerte) -->
+    <!-- Hand states for RViz/MoveIt. These joints are actively controlled via
+         mia_joint_trajectory_controller, so they must not be passive joints. -->
     <group_state name="hand_open" group="mia_hand">
-      <joint name="j_thumb_fle" value="0.1"/>
+      <joint name="j_thumb_fle" value="0.0"/>
       <joint name="j_thumb_opp" value="-0.4"/>
-      <joint name="j_index_fle" value="0"/>
-      <joint name="j_mrl_fle"  value="0.1"/>
+      <joint name="j_index_fle" value="0.0"/>
+      <joint name="j_mrl_fle"  value="0.0"/>
     </group_state>
+    <!-- Collision-free closing pose.
+         The previous 1.0 / -0.1 / 1.0 / 1.0 pose closes the hand too far in
+         MoveIt's collision model: thumb_fle intersects index_sensor /
+         middle_sensor. This pose still curls the fingers, but keeps the thumb
+         slightly opened / rotated away so Plan & Execute can run without
+         disabling those collisions. -->
     <group_state name="hand_close" group="mia_hand">
-      <joint name="j_thumb_fle" value="0.3"/>
-      <joint name="j_thumb_opp" value="-0.1"/>
-      <joint name="j_index_fle" value="0.5"/>
-      <joint name="j_mrl_fle"  value="0.5"/>
+      <joint name="j_thumb_fle" value="0.45"/>
+      <joint name="j_thumb_opp" value="-0.45"/>
+      <joint name="j_index_fle" value="0.85"/>
+      <joint name="j_mrl_fle"  value="0.85"/>
     </group_state>
-    <passive_joint name="j_thumb_fle"/>
-    <passive_joint name="j_index_fle"/>
-    <passive_joint name="j_mrl_fle"/>
-    <passive_joint name="j_thumb_opp"/>
     <!--VIRTUAL JOINT - Purpose - this element defines a virtual joint between a robot link and an external frame of reference (considered fixed with respect to the robot)-->
     <!--DISABLE COLLISIONS - By default it is assumed that any link of the robot could potentially come into collision with any other link in the robot. This tag disables collision checking between a specified pair of links. -->
@@ -78,4 +81,8 @@
     <disable_collisions link1="wrist_2_link" link2="wrist_3_link" reason="Adjacent" />
     <disable_collisions link1="index_fle" link2="index_sensor" reason="Adjacent"/>
+    <!-- MIA hand internal collision matrix.
+         The index_sensor/thumb_fle and middle_sensor/thumb_fle collisions are
+         intentionally NOT disabled here. Instead, the hand_close named state
+         above is chosen so the hand closes without self-collision. -->
     <disable_collisions link1="little_fle" link2="palm" reason="Adjacent"/>
     <disable_collisions link1="index_fle" link2="palm" reason="Adjacent"/>
