Commit message: 1st benutzbare version

File: code/manipulator_description/urdf/manipulator_mobile.urdf.xacro (robot description, xacro)
@@ -61,4 +61,5 @@
   <xacro:arg name="simulation_controllers" default="" />
   <xacro:arg name="ros_namespace" default="" />
+  <xacro:arg name="lock_base_tilt" default="true" />
   <xacro:arg name="initial_positions_file" default="$(find ur_description)/config/initial_positions.yaml"/>
   <xacro:property name="initial_positions_file" default="$(arg initial_positions_file)"/>
@@ -83,4 +84,38 @@
     fix_wheel_joints="true">
   </xacro:ranger_air_description>
+  <xacro:if value="$(arg lock_base_tilt)">
+    <!-- Anti-tip stabilisation for the mobile Gazebo setup.
+         The mobile base is moved by gz-sim-velocity-control-system via /cmd_vel,
+         so we do not need Gazebo to solve roll/pitch dynamics for the root link.
+         Marking ranger_base_link as kinematic prevents the complete robot from
+         tipping over, while x/y/yaw motion through /cmd_vel still works.
+         The hidden ballast link is an additional fallback for Gazebo versions that
+         ignore <kinematic> from URDF conversion: it lowers the combined centre of
+         mass and makes roll/pitch numerically very hard to excite. -->
+    <gazebo reference="ranger_base_link">
+      <gravity>false</gravity>
+      <kinematic>true</kinematic>
+      <self_collide>false</self_collide>
+    </gazebo>
+    <link name="anti_tip_ballast_link">
+      <inertial>
+        <origin xyz="0 0 -0.20" rpy="0 0 0"/>
+        <mass value="250.0"/>
+        <inertia
+          ixx="5000.0" ixy="0.0" ixz="0.0"
+          iyy="5000.0" iyz="0.0"
+          izz="5000.0"/>
+      </inertial>
+    </link>
+    <joint name="anti_tip_ballast_joint" type="fixed">
+      <parent link="ranger_base_link"/>
+      <child link="anti_tip_ballast_link"/>
+      <origin xyz="0 0 0" rpy="0 0 0"/>
+    </joint>
+    <gazebo reference="anti_tip_ballast_link">
+      <visualize>false</visualize>
+      <self_collide>false</self_collide>
+    </gazebo>
+  </xacro:if>
   <!-- UR chassis mounted on the Ranger Air base -->
   <xacro:ur_chasis

File: code/manipulator_description/urdf/mia_hand.ros2_control.xacro (robot description, xacro)
@@ -38,5 +38,5 @@
       <joint name="${prefix}j_thumb_fle">
         <command_interface name="position">
-          <param name="min">0.0</param>
+          <param name="min">-0.001</param>
           <param name="max">1.2</param>
         </command_interface>
@@ -46,5 +46,5 @@
         </command_interface>
         <state_interface name="position">
-          <param name="initial_value">0.0</param>
+          <param name="initial_value">0.01</param>
         </state_interface>
         <state_interface name="velocity">
@@ -55,5 +55,5 @@
       <joint name="${prefix}j_index_fle">
         <command_interface name="position">
-          <param name="min">0.0</param>
+          <param name="min">-0.001</param>
           <param name="max">1.2</param>
         </command_interface>
@@ -63,5 +63,5 @@
         </command_interface>
         <state_interface name="position">
-          <param name="initial_value">0.0</param>
+          <param name="initial_value">0.01</param>
         </state_interface>
         <state_interface name="velocity">
@@ -72,5 +72,5 @@
       <joint name="${prefix}j_mrl_fle">
         <command_interface name="position">
-          <param name="min">0.0</param>
+          <param name="min">-0.001</param>
           <param name="max">1.2</param>
         </command_interface>
@@ -80,5 +80,5 @@
         </command_interface>
         <state_interface name="position">
-          <param name="initial_value">0.0</param>
+          <param name="initial_value">0.01</param>
         </state_interface>
         <state_interface name="velocity">

File: code/manipulator_description/urdf/mia_hand.urdf.xacro (robot description, xacro)
@@ -10,5 +10,5 @@
       *origin">
     <!-- Importing URDF macro related to the specified laterality -->
-    <xacro:include filename="$(find mia_hand_description)/urdf/mia_hand_${laterality}.urdf.xacro"/>
+    <xacro:include filename="$(find manipulator_description)/urdf/mia_hand_${laterality}.urdf.xacro"/>
     <!-- Loading proper URDF, depending on the specified laterality -->
     <xacro:if value="${'right' == laterality}">

File: code/manipulator_description/urdf/ur_chasis.xacro (robot description, xacro)
@@ -16,8 +16,13 @@
         </geometry>
       </collision>
+      <!-- Stabilised inertial model:
+           The old centre of mass was 0.5 m above the chassis link, which made
+           the mobile manipulator very top-heavy in Gazebo. The visual/collision
+           geometry is unchanged; only the hidden inertial model is moved down
+           and made numerically stiff against roll/pitch. -->
       <inertial>
-        <origin xyz="0 0 0.5" rpy="0 0 0"/>
-        <mass value="20"/>
-        <inertia ixx="100"  ixy="0"  ixz="0" iyy="100" iyz="0" izz="100" />
+        <origin xyz="0 0 0.12" rpy="0 0 0"/>
+        <mass value="60"/>
+        <inertia ixx="300"  ixy="0"  ixz="0" iyy="300" iyz="0" izz="300" />
       </inertial>
     </link>

File: code/manipulator_ur_moveit_config/srdf/manipulator_macro.srdf.xacro (robot description, xacro)
@@ -67,4 +67,10 @@
       <joint name="j_mrl_fle"  value="0.85"/>
     </group_state>
+    <group_state name="hand_nice_gesture" group="mia_hand">
+      <joint name="j_thumb_fle" value="0.22"/>
+      <joint name="j_thumb_opp" value="0"/>
+      <joint name="j_index_fle" value="1.21"/>
+      <joint name="j_mrl_fle"  value="0.92"/>
+    </group_state>
     <!--VIRTUAL JOINT - Purpose - this element defines a virtual joint between a robot link and an external frame of reference (considered fixed with respect to the robot)-->
     <!--DISABLE COLLISIONS - By default it is assumed that any link of the robot could potentially come into collision with any other link in the robot. This tag disables collision checking between a specified pair of links. -->
