Commit message: added camera sensor with manual gazebo plugin

File: code/manipulator_description/urdf/_d435.urdf.xacro (robot description, xacro)
@@ -3,5 +3,5 @@
 License: Apache 2.0. See LICENSE file in root directory.
 Copyright(c) 2017 Intel Corporation. All Rights Reserved
-This is the URDF model for the Intel RealSense 430 camera, in its
+This is the URDF model for the Intel RealSense 435 camera, in its
 aluminum peripherial evaluation case.
 -->
@@ -77,4 +77,37 @@
       </inertial>
     </link>
+ <!-- Gazebo simulated RGB-D camera. uses same frame for depth and color camera which is technically not correct but practically irrelevant-->
+      <gazebo reference="${name}_simulated_color_frame">
+        <sensor name="${name}_rgbd_sensor" type="rgbd_camera">
+          <always_on>true</always_on>
+          <update_rate>30</update_rate>
+          <visualize>true</visualize>
+          <!-- Base topic for the simulated RGB-D sensor -->
+          <topic>${name}/rgbd</topic>
+          <gz_frame_id>${name}_simulated_color_frame</gz_frame_id>
+          <camera>
+            <!-- Approximate D435 RGB horizontal field of view -->
+            <horizontal_fov>1.211</horizontal_fov>
+            <image>
+              <width>640</width>
+              <height>480</height>
+              <format>R8G8B8</format>
+            </image>
+            <clip>
+              <near>0.1</near>
+              <far>10.0</far>
+            </clip>
+          </camera>
+          <!-- Approximate D435 stereo baseline -->
+          <baseline>0.05</baseline>
+        </sensor>
+      </gazebo>
+      <!-- simulated camera color joints and links. exists because real one does not exist if "use_nominal_extrinsics" is set to false. (the real one is wrong anyway for for a gazebo simulated camera)-->
+      <joint name="${name}_simulated_color_joint" type="fixed">
+        <origin xyz="0 ${d435_cam_depth_to_color_offset} 0" rpy="${M_PI} ${M_PI} 0" />
+        <parent link="${name}_link" />
+        <child link="${name}_simulated_color_frame" />
+      </joint>
+      <link name="${name}_simulated_color_frame"/>
     <!-- Use the nominal extrinsics between camera frames if the calibrated extrinsics aren't being published. e.g. running the device in simulation  -->
     <xacro:if value="${use_nominal_extrinsics}">
